Commit message: kalman filter implementation

File: src/bumperbot_description/urdf/bumperbot.urdf.xacro (robot description, xacro)
@@ -162,3 +162,37 @@
         <origin xyz="-0.04755 0 -0.0275" rpy="0 0 0"/>
     </joint>
+    <!-- IMU link -->
+    <link name="imu_link">
+        <!-- For our purpose, imu's inertial and mass values are not that important. These were added to ensure gazebo loads the model correctly. -->
+        <!-- These values were exported from solidworks -->
+        <inertial>
+        <origin xyz="-0.00552433659106688 0.000168210391520346 0.000514000497342681" rpy="0 0 0" />
+        <mass value="0.000528415362211671" />
+        <inertia ixx="1.46176048428261E-08" ixy="1.40015117949421E-10" ixz="-1.99633872937403E-12"
+                iyy="8.59662482954888E-09" iyz="7.52375112767959E-12"
+                izz="2.30279421279312E-08" />
+        </inertial>
+        <visual>
+        <origin xyz="0 0 0" rpy="0 0 0" />
+        <geometry>
+            <mesh filename="package://bumperbot_description/meshes/imu_link.STL" />
+        </geometry>
+        <material name="">
+            <color rgba="0.792156862745098 0.819607843137255 0.933333333333333 1" />
+        </material>
+        </visual>
+        <collision>
+        <origin xyz="0 0 0" rpy="0 0 0" />
+        <geometry>
+            <mesh filename="package://bumperbot_description/meshes/imu_link.STL" />
+        </geometry>
+        </collision>
+  </link>
+  <!-- Joint connecting IMU link to base link -->
+  <joint name="imu_joint" type="fixed">
+    <origin xyz="0 0 0.0698986241758014" rpy="0 0 0" />
+    <parent link="base_link" />
+    <child link="imu_link" />
+    <axis xyz="0 0 0" />
+  </joint>
 </robot>

File: src/bumperbot_description/urdf/bumperbot_gazebo.urdf.xacro (robot description, xacro)
@@ -45,4 +45,6 @@
         <parameters>$(find bumperbot_controller)/config/bumperbot_controllers.yaml</parameters>
       </plugin>
+      <plugin filename="ignition-gazebo-imu-system" name="ignition::gazebo::systems::Imu">
+      </plugin>
     </xacro:if>
   </gazebo>
@@ -53,5 +55,69 @@
         <parameters>$(find bumperbot_controller)/config/bumperbot_controllers.yaml</parameters>
       </plugin>
+      <plugin filename="gz-sim-imu-system" name="gz::sim::systems::Imu">
+      </plugin>
     </xacro:unless>
   </gazebo>
+  <!-- This section defines an IMU sensor attached to imu_link in Gazebo -->
+  <gazebo reference="imu_link">
+    <sensor name="imu" type="imu">
+      <!-- Ensure the sensor is always active -->
+      <always_on>true</always_on>
+      <!-- Sensor update rate in Hz (100 measurements per second) -->
+      <update_rate>100</update_rate>
+      <!-- Frame ID used for publishing IMU data -->
+      <gz_frame_id>imu_link</gz_frame_id>
+      <!-- Gazebo topic on which IMU data is published -->
+      <topic>imu</topic>
+      <imu>
+        <!-- Gaussian noise applied independently to each gyro axis -->
+        <angular_velocity>
+          <x>
+            <noise type="gaussian">
+              <!-- Zero-mean white noise -->
+              <mean>0.0</mean>
+              <!-- Standard deviation based on IMU gyro noise characteristics -->
+              <stddev>2e-4</stddev>
+            </noise>
+          </x>
+          <y>
+            <noise type="gaussian">
+              <mean>0.0</mean>
+              <stddev>2e-4</stddev>
+            </noise>
+          </y>
+          <z>
+            <noise type="gaussian">
+              <mean>0.0</mean>
+              <!-- Angular velocity noise is smaller than linear acceleration
+                  (consistent with typical IMU datasheets) -->
+              <stddev>2e-4</stddev>
+            </noise>
+          </z>
+        </angular_velocity>
+        <!-- Higher noise compared to angular velocity, as expected for accelerometers -->
+        <linear_acceleration>
+          <x>
+            <noise type="gaussian">
+              <mean>0.0</mean>
+              <!-- Standard deviation reflects accelerometer noise -->
+              <stddev>1.7e-2</stddev>
+            </noise>
+          </x>
+          <y>
+            <noise type="gaussian">
+              <mean>0.0</mean>
+              <stddev>1.7e-2</stddev>
+            </noise>
+          </y>
+          <z>
+            <noise type="gaussian">
+              <mean>0.0</mean>
+              <stddev>1.7e-2</stddev>
+            </noise>
+          </z>
+        </linear_acceleration>
+      </imu>
+    </sensor>
+  </gazebo>
 </robot>

Commit message: mapping

File: src/bumperbot_description/urdf/bumperbot.urdf.xacro (robot description, xacro)
@@ -24,4 +24,5 @@
                 <mesh filename="package://bumperbot_description/meshes/base_link.STL"/>
             </geometry>
+            <material name="black"/>
         </visual>
         <!-- Collision geometry for physics simulation. Same mesh.-->
@@ -54,4 +55,5 @@
                 <mesh filename="package://bumperbot_description/meshes/wheel_right_link.STL"/>
             </geometry>
+            <material name="blue"/>
         </visual>
         <!-- Collision geometry for physics simulation. Sphere approximation of wheel -->
@@ -87,4 +89,5 @@
                 <mesh filename="package://bumperbot_description/meshes/wheel_left_link.STL"/>
             </geometry>
+            <material name="blue"/>
         </visual>
         <!-- Collision geometry for physics simulation. Sphere approximation of wheel -->
@@ -118,4 +121,5 @@
                 <mesh filename="package://bumperbot_description/meshes/caster_front_link.STL"/>
             </geometry>
+            <material name="silver"/>
         </visual>
         <!-- Collision geometry for physics simulation. Sphere approximation of caster -->
@@ -147,4 +151,5 @@
                 <mesh filename="package://bumperbot_description/meshes/caster_rear_link.STL"/>
             </geometry>
+            <material name="silver"/>
         </visual>
         <!-- Collision geometry for physics simulation. Sphere approximation of caster -->
@@ -181,4 +186,5 @@
             <color rgba="0.792156862745098 0.819607843137255 0.933333333333333 1" />
         </material>
+        <material name="blue"/>
         </visual>
         <collision>
@@ -196,3 +202,43 @@
     <axis xyz="0 0 0" />
   </joint>
+    <link name="laser_link">
+    <inertial>
+      <origin xyz="-0.011945780406062 -0.000381929217680526 -0.0170649378129477" rpy="0 0 0" />
+      <mass value="0.073084435549317" />
+      <inertia ixx="1.96074931730795E-05" ixy="-3.62091076640009E-07" ixz="4.28230084046735E-07"
+               iyy="2.40983835136327E-05" iyz="1.50180909250652E-08"
+               izz="4.14184164228595E-05" />
+    </inertial>
+    <visual>
+      <origin xyz="0 0 0" rpy="0 0 0" />
+      <geometry>
+        <mesh filename="package://bumperbot_description/meshes/laser_link.STL" />
+      </geometry>
+      <material name="dark_grey"/>
+    </visual>
+    <collision>
+      <origin xyz="0 0 0" rpy="0 0 0" />
+      <geometry>
+        <mesh filename="package://bumperbot_description/meshes/laser_link.STL" />
+      </geometry>
+    </collision>
+  </link>
+  <joint name="laser_joint" type="fixed">
+    <origin xyz="-0.0050526 -0.0023221 0.1208" rpy="0 0 3.14" />
+    <parent link="base_link" />
+    <child link="laser_link" />
+    <axis xyz="0 0 0" />
+  </joint>
+  <material name="blue">
+  <color rgba="0 0 1 1"/>
+  </material>
+  <material name="black">
+    <color rgba="0 0 0 1"/>
+  </material>
+  <material name="silver">
+    <color rgba="0.79 0.82 0.93 1"/>
+  </material>
+  <material name="dark_grey">
+    <color rgba="0.3 0.3 0.3 1"/>
+  </material>
 </robot>

File: src/bumperbot_description/urdf/bumperbot_gazebo.urdf.xacro (robot description, xacro)
@@ -47,4 +47,7 @@
       <plugin filename="ignition-gazebo-imu-system" name="ignition::gazebo::systems::Imu">
       </plugin>
+       <plugin filename="ignition-gazebo-sensors-system" name="ignition::gazebo::systems::Sensors">
+        <render_engine>ogre2</render_engine>
+      </plugin>
     </xacro:if>
   </gazebo>
@@ -56,4 +59,7 @@
       </plugin>
       <plugin filename="gz-sim-imu-system" name="gz::sim::systems::Imu">
+      </plugin>
+            <plugin filename="gz-sim-sensors-system" name="gz::sim::systems::Sensors">
+        <render_engine>ogre2</render_engine>
       </plugin>
     </xacro:unless>
@@ -121,3 +127,32 @@
     </sensor>
   </gazebo>
+  <gazebo reference="laser_link">
+    <sensor name="lidar" type="gpu_lidar">
+      <always_on>true</always_on>
+      <visualize>true</visualize>
+      <topic>scan</topic>
+      <update_rate>5</update_rate>
+      <gz_frame_id>laser_link</gz_frame_id>
+      <lidar>
+        <scan>
+          <horizontal>
+            <samples>360</samples>
+            <resolution>1.00000</resolution>
+            <min_angle>0.000000</min_angle>
+            <max_angle>6.280000</max_angle>
+          </horizontal>
+        </scan>
+        <range>
+          <min>0.120000</min>
+          <max>12.0</max>
+          <resolution>0.02</resolution>
+        </range>
+        <noise>
+          <type>gaussian</type>
+          <mean>0.0</mean>
+          <stddev>0.01</stddev>
+        </noise>
+      </lidar>
+    </sensor>
+  </gazebo>
 </robot>
